Commit message: reorganized

File: carter_description/urdf/carter.urdf (robot description, URDF)
Before this commit: robot carter, 3 links, 1 joints
Joints:
- removed joint base
- added joint wheel_l_joint: type continuous, parent base_link, child wheel_l, origin xyz=0 0 0 rpy=0 0 0, axis 1 0 0
- added joint wheel_r_joint: type continuous, parent base_link, child wheel_r, origin xyz=0.1242 -0.000183 0.009979 rpy=0 0 0, axis 1 0 0

Commit message: commits

File: carter_description/urdf/carter.urdf (robot description, URDF)
Before this commit: robot carter, 3 links, 2 joints
Links:
- removed link wheel_l
- removed link wheel_r
- added link wheel_left_link; visual mesh filename=file:/home/andrea/catkin_ws/src/carter/carter_description/m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 scale=0.001 0.001 0.001
- added link wheel_rear_link; visual mesh filename=file:/home/andrea/catkin_ws/src/carter/carter_description/m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 scale=0.001 0.001 0.001
- added link wheel_right_link; visual mesh filename=file:/home/andrea/catkin_ws/src/carter/carter_description/m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 scale=0.001 0.001 0.001
Joints:
- removed joint wheel_l_joint
- removed joint wheel_r_joint
- added joint wheel_left_joint: type continuous, parent base_link, child wheel_left_link, origin xyz=-0.000076 0.1242 0.009999 rpy=-1.5708 0 0, axis 0 0 1
- added joint wheel_rear_joint: type fixed, parent base_link, child wheel_rear_link, origin xyz=0 0 0 rpy=0 0 0, axis 0 0 0
- added joint wheel_right_joint: type continuous, parent base_link, child wheel_right_link, origin xyz=-0.000076 -0.1242 0.009999 rpy=-1.5708 0 0, axis 0 0 1

Commit message: commits

File: carter_description/urdf/carter.urdf (robot description, URDF)
Before this commit: robot carter, 4 links, 3 joints
Joints:
- joint wheel_rear_joint: axis 0 0 0 -> (none)

Commit message: major changes

File: carter_description/urdf/carter.urdf (robot description, URDF)
Before this commit: robot carter, 4 links, 3 joints
Links:
- added link imu_link
- added link mag_link
Joints:
- added joint imu_joint: type fixed, parent base_link, child imu_link, origin xyz=0 0 0 rpy=0 0 0
- added joint mag_joint: type fixed, parent base_link, child mag_link, origin xyz=0 0 0 rpy=0 0 0
